File: solar/power-hop-hardware-main/battery-protection.kicad_sch (KiCad schematic)
At the start: 11 parts, among them Q5 SSM3J355R,LF, Q6 EFC3J018NUZTDG, U11 BQ298000

Commit message: Remapped Q5 and rerouted traces
Connections:
- net BAT_N: now also Q5.1 (G); no longer Q5.2 (G)
- net BAT_P: now also Q5.2 (S); no longer Q5.3 (S)
- net BAT_P_POL: now also Q5.3 (D); no longer Q5.1 (D)
